File: Hardware/Micro_Bit_Control_Bit.brd (EAGLE design)
At the start: 152.4 x 50.8 mm, 39 parts, among them J1 Pokehome, J2 Pokehome, J3 Pokehome, J4 Pokehome, J5 Pokehome, J6 Pokehome, J7 Pokehome, J8 Pokehome, J9 QWIIC_RA, U2 micro:bit

Commit message: Updated contro bit text silk to match other boards
Parts:
- moved U$4 5.08 mm to (64.0, 2.86)
- moved U$5 4.19 mm to (87.8, 30.3)
- moved LOGO1 1.91 mm to (89.2, 2.60)
Changed lines of the file:
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@@
 <attribute name="PROD_ID" value="CONN-13512" x="146.05" y="41.275" size="1.778" layer="28" font="vector" ratio="15" rot="MR270" display="off"/>
 </element>
-<element name="LOGO1" library="SparkFun-Aesthetics" package="SFE_LOGO_FLAME_.2" value="SFE_LOGO_FLAME.2_INCH" x="91.15425" y="2.4765" smashed="yes"/>
+<element name="LOGO1" library="SparkFun-Aesthetics" package="SFE_LOGO_FLAME_.2" value="SFE_LOGO_FLAME.2_INCH" x="89.24925" y="2.6035" smashed="yes"/>
 <element name="LOGO2" library="SparkFun-Aesthetics" package="OSHW-LOGO-L" value="OSHW-LOGOL" x="76.2" y="25.4" smashed="yes" rot="MR0"/>
 <element name="LOGO3" library="SparkFun-Aesthetics" package="SFE_LOGO_NAME_FLAME_.3" value="SFE_LOGO_NAME_FLAME.3_INCH" x="92.71" y="34.29" smashed="yes" rot="MR0"/>
@@
 <attribute name="VALUE" x="95.25" y="15.24" size="1.27" layer="27" font="vector"/>
 </element>
-<element name="U$4" library="Micro_Bit_Parts" package="LOGO-CONTROLBIT" value="LOGO-CONTROLBIT" x="58.95975" y="2.8575" smashed="yes"/>
-<element name="U$5" library="Micro_Bit_Parts" package="LOGO-CONTROLBIT" value="LOGO-CONTROLBIT" x="91.97975" y="30.4165" smashed="yes" rot="MR0"/>
+<element name="U$4" library="Micro_Bit_Parts" package="LOGO-CONTROLBIT" value="LOGO-CONTROLBIT" x="64.03975" y="2.8575" smashed="yes"/>
+<element name="U$5" library="Micro_Bit_Parts" package="LOGO-CONTROLBIT" value="LOGO-CONTROLBIT" x="87.78875" y="30.2895" smashed="yes" rot="MR0"/>
 <element name="J9" library="SparkFun-Connectors" package="JST04_1MM_RA" value="QWIIC_RA" x="126.492" y="45.593" smashed="yes" rot="MR180">
 <attribute name="NAME" x="126.508" y="41.02666875" size="0.6096" layer="26" rot="MR180"/>

Commit message: Adding test points
Parts:
- added TP1, TP10, TP11, TP12, TP13, TP2, TP3, TP4, TP5, TP6, TP7, TP8, TP9: (no value), SparkFun-Connectors:PAD.03X.03
- moved LOGO2 1.27 mm to (76.2, 24.1)
Connections:
- net 3.3V: now also TP1.P$1
- net BTN_A: now also TP12.P$1
- net BTN_B: now also TP9.P$1
- net BTN_DN: now also TP10.P$1
- net BTN_L: now also TP11.P$1
- net BTN_P12: now also TP8.P$1
- net BTN_P16: now also TP6.P$1
- net BTN_R: now also TP7.P$1
- net BTN_UP: now also TP13.P$1
- net GND: now also TP2.P$1, TP3.P$1
- net SCL: now also TP5.P$1
- net SDA: now also TP4.P$1
Routing:
- net 3.3V: track 101.5 -> 126.6 mm, vias 1 -> 2
- net SDA: track 77.3 -> 96.4 mm, vias 1 -> 2
- net BTN_P16: track 53.3 -> 71.6 mm, vias 0 -> 1
- net SCL: track 84.7 -> 102.7 mm, vias 1 -> 2
- net BTN_UP: track 29.0 -> 42.1 mm, vias 0 -> 1
- net BTN_DN: track 38.6 -> 50.1 mm, vias 0 -> 1
- net BTN_R: track 60.0 -> 71.5 mm, vias 0 -> 1
- net BTN_L: track 42.3 -> 53.8 mm, vias 0 -> 1
- net BTN_P12: track 61.7 -> 70.7 mm, vias 0 -> 1
- net BTN_B: track 60.8 -> 69.7 mm, vias 0 -> 1
- net BTN_A: track 56.6 -> 64.3 mm, vias 0 -> 1
Changed lines of the file:
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@@
 </element>
 <element name="LOGO1" library="SparkFun-Aesthetics" package="SFE_LOGO_FLAME_.2" value="SFE_LOGO_FLAME.2_INCH" x="89.24925" y="2.6035" smashed="yes"/>
-<element name="LOGO2" library="SparkFun-Aesthetics" package="OSHW-LOGO-L" value="OSHW-LOGOL" x="76.2" y="25.4" smashed="yes" rot="MR0"/>
+<element name="LOGO2" library="SparkFun-Aesthetics" package="OSHW-LOGO-L" value="OSHW-LOGOL" x="76.2" y="24.13" smashed="yes" rot="MR0"/>
 <element name="LOGO3" library="SparkFun-Aesthetics" package="SFE_LOGO_NAME_FLAME_.3" value="SFE_LOGO_NAME_FLAME.3_INCH" x="92.71" y="34.29" smashed="yes" rot="MR0"/>
 <element name="FD1" library="SparkFun-Aesthetics" package="FIDUCIAL-MICRO" value="FIDUCIALUFIDUCIAL" x="2.54" y="49.53" smashed="yes"/>
@@
 </element>
 <element name="U$2" library="SparkFun-Aesthetics" package="QWIIC_5MM" value="" x="126.7714" y="43.6372" smashed="yes" rot="MR0"/>
+<element name="TP1" library="SparkFun-Connectors" package="PAD.03X.03" value="" x="86.36" y="29.21" smashed="yes" rot="MR90"/>
+<element name="TP2" library="SparkFun-Connectors" package="PAD.03X.03" value="" x="88.9" y="29.21" smashed="yes" rot="MR90"/>
+<element name="TP3" library="SparkFun-Connectors" package="PAD.03X.03" value="" x="58.42" y="29.21" smashed="yes" rot="MR90"/>
+<element name="TP4" library="SparkFun-Connectors" package="PAD.03X.03" value="" x="83.82" y="29.21" smashed="yes" rot="MR90"/>
+<element name="TP5" library="SparkFun-Connectors" package="PAD.03X.03" value="" x="81.28" y="29.21" smashed="yes" rot="MR90"/>
+<element name="TP6" library="SparkFun-Connectors" package="PAD.03X.03" value="" x="78.74" y="29.21" smashed="yes" rot="MR90"/>
+<element name="TP7" library="SparkFun-Connectors" package="PAD.03X.03" value="" x="76.2" y="29.21" smashed="yes" rot="MR90"/>
+<element name="TP8" library="SparkFun-Connectors" package="PAD.03X.03" value="" x="73.66" y="29.21" smashed="yes" rot="MR90"/>
+<element name="TP9" library="SparkFun-Connectors" package="PAD.03X.03" value="" x="71.12" y="29.21" smashed="yes" rot="MR90"/>
+<element name="TP10" library="SparkFun-Connectors" package="PAD.03X.03" value="" x="68.58" y="29.21" smashed="yes" rot="MR90"/>
+<element name="TP11" library="SparkFun-Connectors" package="PAD.03X.03" value="" x="66.04" y="29.21" smashed="yes" rot="MR90"/>
+<element name="TP12" library="SparkFun-Connectors" package="PAD.03X.03" value="" x="63.5" y="29.21" smashed="yes" rot="MR90"/>
+<element name="TP13" library="SparkFun-Connectors" package="PAD.03X.03" value="" x="60.96" y="29.21" smashed="yes" rot="MR90"/>
 </elements>
 <signals>
@@
 <wire x1="53.975" y1="17.98" x2="53.975" y2="15.24" width="0.254" layer="1"/>
 <wire x1="55.245" y1="17.98" x2="55.245" y2="15.24" width="0.254" layer="1"/>
+<contactref element="TP13" pad="P$1"/>
+<wire x1="56.515" y1="17.98" x2="56.515" y2="20.447" width="0.254" layer="1"/>
+<via x="56.515" y="20.447" extent="1-16" drill="0.508"/>
+<wire x1="56.515" y1="20.447" x2="56.515" y2="24.765" width="0.254" layer="16"/>
+<wire x1="56.515" y1="24.765" x2="60.96" y2="29.21" width="0.254" layer="16"/>
 </signal>
 <signal name="BTN_L">
@@
 <wire x1="64.135" y1="17.98" x2="64.135" y2="15.24" width="0.254" layer="1"/>
 <wire x1="65.405" y1="17.98" x2="65.405" y2="15.24" width="0.254" layer="1"/>
+<contactref element="TP11" pad="P$1"/>
+<wire x1="66.675" y1="17.98" x2="66.675" y2="20.955" width="0.254" layer="1"/>
+<wire x1="66.675" y1="20.955" x2="66.04" y2="21.59" width="0.254" layer="1"/>
+<via x="66.04" y="21.59" extent="1-16" drill="0.508"/>
+<wire x1="66.04" y1="21.59" x2="66.04" y2="29.21" width="0.254" layer="16"/>
 </signal>
 <signal name="BTN_R">
@@
 <wire x1="41.148" y1="6.985" x2="70.993" y2="6.985" width="0.254" layer="1"/>
 <wire x1="75.184" y1="11.176" x2="75.184" y2="15.24" width="0.254" layer="1"/>
+<contactref element="TP7" pad="P$1"/>
+<wire x1="76.835" y1="17.98" x2="76.835" y2="20.066" width="0.254" layer="1"/>
+<via x="76.835" y="20.066" extent="1-16" drill="0.508"/>
+<wire x1="76.835" y1="20.066" x2="76.2" y2="20.701" width="0.254" layer="16"/>
+<wire x1="76.2" y1="20.701" x2="76.2" y2="29.21" width="0.254" layer="16"/>
 </signal>
 <signal name="BTN_DN">
@@
 <wire x1="64.897" y1="8.128" x2="67.945" y2="11.176" width="0.254" layer="1"/>
 <wire x1="41.91" y1="8.128" x2="64.897" y2="8.128" width="0.254" layer="1"/>
+<contactref element="TP10" pad="P$1"/>
+<wire x1="67.945" y1="17.98" x2="67.945" y2="20.955" width="0.254" layer="1"/>
+<wire x1="67.945" y1="20.955" x2="68.58" y2="21.59" width="0.254" layer="1"/>
+<via x="68.58" y="21.59" extent="1-16" drill="0.508"/>
+<wire x1="68.58" y1="21.59" x2="68.58" y2="29.21" width="0.254" layer="16"/>
 </signal>
 <signal name="BTN_P16">
@@
 <wire x1="83.693" y1="20.574" x2="83.185" y2="20.066" width="0.254" layer="1"/>
 <wire x1="83.185" y1="20.066" x2="83.185" y2="17.98" width="0.254" layer="1"/>
+<contactref element="TP6" pad="P$1"/>
+<wire x1="83.185" y1="17.98" x2="83.185" y2="15.367" width="0.254" layer="1"/>
+<via x="83.185" y="15.367" extent="1-16" drill="0.508"/>
+<wire x1="83.185" y1="15.367" x2="78.74" y2="19.812" width="0.254" layer="16"/>
+<wire x1="78.74" y1="19.812" x2="78.74" y2="29.21" width="0.254" layer="16"/>
 </signal>
 <signal name="BTN_P12">
@@
 <wire x1="125.857" y1="12.192" x2="126.365" y2="12.7" width="0.254" layer="1"/>
 <wire x1="126.365" y1="12.7" x2="126.365" y2="14.39" width="0.254" layer="1"/>
+<contactref element="TP8" pad="P$1"/>
+<wire x1="73.66" y1="29.21" x2="73.66" y2="21.082" width="0.254" layer="16"/>
+<wire x1="73.66" y1="21.082" x2="73.025" y2="20.447" width="0.254" layer="16"/>
+<via x="73.025" y="20.447" extent="1-16" drill="0.508"/>
 </signal>
 <signal name="3.3V">
@@
 <wire x1="88.265" y1="17.98" x2="88.265" y2="15.24" width="0.508" layer="1"/>
 <wire x1="89.535" y1="17.98" x2="89.535" y2="15.24" width="0.508" layer="1"/>
+<contactref element="TP1" pad="P$1"/>
+<wire x1="86.36" y1="29.21" x2="84.582" y2="30.988" width="0.254" layer="16"/>
+<wire x1="84.582" y1="30.988" x2="81.153" y2="30.988" width="0.254" layer="16"/>
+<wire x1="81.153" y1="30.988" x2="80.01" y2="29.845" width="0.254" layer="16"/>
+<wire x1="80.01" y1="29.845" x2="80.01" y2="24.13" width="0.254" layer="16"/>
+<wire x1="86.995" y1="15.24" x2="86.995" y2="17.145" width="0.254" layer="16"/>
+<wire x1="86.995" y1="17.145" x2="80.01" y2="24.13" width="0.254" layer="16"/>
+<via x="86.995" y="15.24" extent="1-16" drill="0.508"/>
 </signal>
 <signal name="GND">
@@
 <via x="66.04" y="12.7" extent="1-16" drill="0.508"/>
 <contactref element="J9" pad="1"/>
+<contactref element="TP2" pad="P$1"/>
+<contactref element="TP3" pad="P$1"/>
 </signal>
 <signal name="N$1">
@@
 <wire x1="59.055" y1="21.717" x2="59.055" y2="17.98" width="0.254" layer="1"/>
 <wire x1="106.68" y1="22.86" x2="60.198" y2="22.86" width="0.254" layer="1"/>
+<contactref element="TP12" pad="P$1"/>
+<wire x1="63.5" y1="29.21" x2="60.198" y2="25.908" width="0.254" layer="16"/>
+<wire x1="60.198" y1="25.908" x2="60.198" y2="22.86" width="0.254" layer="16"/>
+<via x="60.198" y="22.86" extent="1-16" drill="0.508"/>
 </signal>
 <signal name="BTN_B">
@@
 <wire x1="115.57" y1="12.7" x2="106.68" y2="21.59" width="0.254" layer="1"/>
 <wire x1="106.68" y1="21.59" x2="72.771" y2="21.59" width="0.254" layer="1"/>
-<wire x1="72.771" y1="21.59" x2="71.9455" y2="20.7645" width="0.254" layer="1"/>
+<wire x1="72.771" y1="21.59" x2="71.755" y2="20.574" width="0.254" layer="1"/>
 <wire x1="71.755" y1="17.98" x2="71.755" y2="20.574" width="0.254" layer="1"/>
-<wire x1="71.755" y1="20.574" x2="71.9455" y2="20.7645" width="0.254" layer="1"/>
+<contactref element="TP9" pad="P$1"/>
+<wire x1="71.12" y1="29.21" x2="71.755" y2="28.575" width="0.254" layer="16"/>
+<wire x1="71.755" y1="28.575" x2="71.755" y2="20.574" width="0.254" layer="16"/>
+<via x="71.755" y="20.574" extent="1-16" drill="0.508"/>
 </signal>
 <signal name="N$7">
@@
 <wire x1="93.345" y1="14.097" x2="93.345" y2="17.98" width="0.254" layer="1"/>
 <wire x1="98.552" y1="8.89" x2="93.345" y2="14.097" width="0.254" layer="1"/>
+<contactref element="TP4" pad="P$1"/>
+<wire x1="83.82" y1="29.21" x2="83.82" y2="27.051" width="0.254" layer="16"/>
+<wire x1="83.82" y1="27.051" x2="93.345" y2="17.526" width="0.254" layer="16"/>
+<wire x1="93.345" y1="17.526" x2="93.345" y2="14.097" width="0.254" layer="16"/>
+<via x="93.345" y="14.097" extent="1-16" drill="0.508"/>
 </signal>
 <signal name="SCL">
 <contactref element="J9" pad="4"/>
 <contactref element="U2" pad="P$33"/>
-<wire x1="92.075" y1="17.98" x2="92.075" y2="13.716" width="0.254" layer="1"/>
+<wire x1="92.075" y1="17.98" x2="92.075" y2="15.621" width="0.254" layer="1"/>
+<wire x1="92.075" y1="15.621" x2="92.075" y2="13.716" width="0.254" layer="1"/>
 <wire x1="98.171" y1="7.62" x2="130.81" y2="7.62" width="0.254" layer="1"/>
 <via x="130.81" y="7.62" extent="1-16" drill="0.508"/>
@@
 <wire x1="127.992" y1="10.438" x2="127.992" y2="45.593" width="0.254" layer="16"/>
 <wire x1="92.075" y1="13.716" x2="98.171" y2="7.62" width="0.254" layer="1"/>
+<contactref element="TP5" pad="P$1"/>
+<via x="92.075" y="15.621" extent="1-16" drill="0.508"/>
+<wire x1="81.28" y1="29.21" x2="81.28" y2="26.416" width="0.254" layer="16"/>
+<wire x1="81.28" y1="26.416" x2="92.075" y2="15.621" width="0.254" layer="16"/>
 </signal>
 </signals>

Commit message: library thing - control bit text device now in SFE aethetics
Parts:
- U$4, U$5: device Micro_Bit_Parts:LOGO-CONTROLBIT -> SparkFun-Aesthetics:LOGO-CONTROLBIT
Changed lines of the file:
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@@
 <attribute name="VALUE" x="95.25" y="15.24" size="1.27" layer="27" font="vector"/>
 </element>
-<element name="U$4" library="Micro_Bit_Parts" package="LOGO-CONTROLBIT" value="LOGO-CONTROLBIT" x="64.03975" y="2.8575" smashed="yes"/>
-<element name="U$5" library="Micro_Bit_Parts" package="LOGO-CONTROLBIT" value="LOGO-CONTROLBIT" x="87.78875" y="30.2895" smashed="yes" rot="MR0"/>
+<element name="U$4" library="SparkFun-Aesthetics" package="LOGO-CONTROLBIT" value="LOGO-CONTROLBIT" x="64.03975" y="2.8575" smashed="yes"/>
+<element name="U$5" library="SparkFun-Aesthetics" package="LOGO-CONTROLBIT" value="LOGO-CONTROLBIT" x="87.78875" y="30.2895" smashed="yes" rot="MR0"/>
 <element name="J9" library="SparkFun-Connectors" package="JST04_1MM_RA" value="QWIIC_RA" x="126.492" y="45.593" smashed="yes" rot="MR180">
 <attribute name="NAME" x="126.508" y="41.02666875" size="0.6096" layer="26" rot="MR180"/>

Commit message: bumped test ppoints to larger size
also rearragned VCC pin over so it wasn't right next to GND, to help avoid accidental jumpers between VCC and GND.
Parts:
- TP1, TP10, TP11, TP12, TP13, TP2, TP3, TP4, TP5, TP6, TP7, TP8, TP9: value (none) -> TEST-POINT3X5; device SparkFun-Connectors:PAD.03X.03 -> SparkFun-Connectors:PAD.03X.05
- moved TP1 5.08 mm to (81.3, 29.2)
- moved TP4 2.54 mm to (86.4, 29.2)
- moved TP5 2.54 mm to (83.8, 29.2)
Routing:
- net 3.3V: track 126.6 -> 117.8 mm
- net SDA: track 96.4 -> 95.3 mm
- net SCL: track 102.7 -> 101.7 mm
Changed lines of the file:
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@@
 </element>
 <element name="U$2" library="SparkFun-Aesthetics" package="QWIIC_5MM" value="" x="126.7714" y="43.6372" smashed="yes" rot="MR0"/>
-<element name="TP1" library="SparkFun-Connectors" package="PAD.03X.03" value="" x="86.36" y="29.21" smashed="yes" rot="MR90"/>
-<element name="TP2" library="SparkFun-Connectors" package="PAD.03X.03" value="" x="88.9" y="29.21" smashed="yes" rot="MR90"/>
-<element name="TP3" library="SparkFun-Connectors" package="PAD.03X.03" value="" x="58.42" y="29.21" smashed="yes" rot="MR90"/>
-<element name="TP4" library="SparkFun-Connectors" package="PAD.03X.03" value="" x="83.82" y="29.21" smashed="yes" rot="MR90"/>
-<element name="TP5" library="SparkFun-Connectors" package="PAD.03X.03" value="" x="81.28" y="29.21" smashed="yes" rot="MR90"/>
-<element name="TP6" library="SparkFun-Connectors" package="PAD.03X.03" value="" x="78.74" y="29.21" smashed="yes" rot="MR90"/>
-<element name="TP7" library="SparkFun-Connectors" package="PAD.03X.03" value="" x="76.2" y="29.21" smashed="yes" rot="MR90"/>
-<element name="TP8" library="SparkFun-Connectors" package="PAD.03X.03" value="" x="73.66" y="29.21" smashed="yes" rot="MR90"/>
-<element name="TP9" library="SparkFun-Connectors" package="PAD.03X.03" value="" x="71.12" y="29.21" smashed="yes" rot="MR90"/>
-<element name="TP10" library="SparkFun-Connectors" package="PAD.03X.03" value="" x="68.58" y="29.21" smashed="yes" rot="MR90"/>
-<element name="TP11" library="SparkFun-Connectors" package="PAD.03X.03" value="" x="66.04" y="29.21" smashed="yes" rot="MR90"/>
-<element name="TP12" library="SparkFun-Connectors" package="PAD.03X.03" value="" x="63.5" y="29.21" smashed="yes" rot="MR90"/>
-<element name="TP13" library="SparkFun-Connectors" package="PAD.03X.03" value="" x="60.96" y="29.21" smashed="yes" rot="MR90"/>
+<element name="TP1" library="SparkFun-Connectors" package="PAD.03X.05" value="TEST-POINT3X5" x="81.28" y="29.21" smashed="yes" rot="MR90"/>
+<element name="TP2" library="SparkFun-Connectors" package="PAD.03X.05" value="TEST-POINT3X5" x="88.9" y="29.21" smashed="yes" rot="MR90"/>
+<element name="TP3" library="SparkFun-Connectors" package="PAD.03X.05" value="TEST-POINT3X5" x="58.42" y="29.21" smashed="yes" rot="MR90"/>
+<element name="TP4" library="SparkFun-Connectors" package="PAD.03X.05" value="TEST-POINT3X5" x="86.36" y="29.21" smashed="yes" rot="MR90"/>
+<element name="TP5" library="SparkFun-Connectors" package="PAD.03X.05" value="TEST-POINT3X5" x="83.82" y="29.21" smashed="yes" rot="MR90"/>
+<element name="TP6" library="SparkFun-Connectors" package="PAD.03X.05" value="TEST-POINT3X5" x="78.74" y="29.21" smashed="yes" rot="MR90"/>
+<element name="TP7" library="SparkFun-Connectors" package="PAD.03X.05" value="TEST-POINT3X5" x="76.2" y="29.21" smashed="yes" rot="MR90"/>
+<element name="TP8" library="SparkFun-Connectors" package="PAD.03X.05" value="TEST-POINT3X5" x="73.66" y="29.21" smashed="yes" rot="MR90"/>
+<element name="TP9" library="SparkFun-Connectors" package="PAD.03X.05" value="TEST-POINT3X5" x="71.12" y="29.21" smashed="yes" rot="MR90"/>
+<element name="TP10" library="SparkFun-Connectors" package="PAD.03X.05" value="TEST-POINT3X5" x="68.58" y="29.21" smashed="yes" rot="MR90"/>
+<element name="TP11" library="SparkFun-Connectors" package="PAD.03X.05" value="TEST-POINT3X5" x="66.04" y="29.21" smashed="yes" rot="MR90"/>
+<element name="TP12" library="SparkFun-Connectors" package="PAD.03X.05" value="TEST-POINT3X5" x="63.5" y="29.21" smashed="yes" rot="MR90"/>
+<element name="TP13" library="SparkFun-Connectors" package="PAD.03X.05" value="TEST-POINT3X5" x="60.96" y="29.21" smashed="yes" rot="MR90"/>
 </elements>
 <signals>
@@
 <wire x1="89.535" y1="17.98" x2="89.535" y2="15.24" width="0.508" layer="1"/>
 <contactref element="TP1" pad="P$1"/>
-<wire x1="86.36" y1="29.21" x2="84.582" y2="30.988" width="0.254" layer="16"/>
-<wire x1="84.582" y1="30.988" x2="81.153" y2="30.988" width="0.254" layer="16"/>
-<wire x1="81.153" y1="30.988" x2="80.01" y2="29.845" width="0.254" layer="16"/>
-<wire x1="80.01" y1="29.845" x2="80.01" y2="24.13" width="0.254" layer="16"/>
 <wire x1="86.995" y1="15.24" x2="86.995" y2="17.145" width="0.254" layer="16"/>
-<wire x1="86.995" y1="17.145" x2="80.01" y2="24.13" width="0.254" layer="16"/>
+<wire x1="86.995" y1="17.145" x2="81.28" y2="22.86" width="0.254" layer="16"/>
 <via x="86.995" y="15.24" extent="1-16" drill="0.508"/>
+<wire x1="81.28" y1="29.21" x2="81.28" y2="22.86" width="0.254" layer="16"/>
 </signal>
 <signal name="GND">
@@
 <wire x1="98.552" y1="8.89" x2="93.345" y2="14.097" width="0.254" layer="1"/>
 <contactref element="TP4" pad="P$1"/>
-<wire x1="83.82" y1="29.21" x2="83.82" y2="27.051" width="0.254" layer="16"/>
-<wire x1="83.82" y1="27.051" x2="93.345" y2="17.526" width="0.254" layer="16"/>
+<wire x1="86.36" y1="29.21" x2="86.36" y2="24.511" width="0.254" layer="16"/>
+<wire x1="86.36" y1="24.511" x2="93.345" y2="17.526" width="0.254" layer="16"/>
 <wire x1="93.345" y1="17.526" x2="93.345" y2="14.097" width="0.254" layer="16"/>
 <via x="93.345" y="14.097" extent="1-16" drill="0.508"/>
@@
 <contactref element="TP5" pad="P$1"/>
 <via x="92.075" y="15.621" extent="1-16" drill="0.508"/>
-<wire x1="81.28" y1="29.21" x2="81.28" y2="26.416" width="0.254" layer="16"/>
-<wire x1="81.28" y1="26.416" x2="92.075" y2="15.621" width="0.254" layer="16"/>
+<wire x1="83.82" y1="29.21" x2="83.82" y2="23.876" width="0.254" layer="16"/>
+<wire x1="83.82" y1="23.876" x2="92.075" y2="15.621" width="0.254" layer="16"/>
 </signal>
 </signals>
