File: Hardware/Production/Micro_Bit_Control_Bit-Panel.brd (EAGLE design)
At the start: 172.5 x 327.4 mm, 306 parts, among them J1 Pokehome, J10 Pokehome, J11 Pokehome, J12 Pokehome, J13 Pokehome, J14 Pokehome, J15 Pokehome, J16 Pokehome, J17 Pokehome, J18 QWIIC_RA, J19 Pokehome, J2 Pokehome, J20 Pokehome, J21 Pokehome, J22 Pokehome, J23 Pokehome, J24 Pokehome, J25 Pokehome, J26 Pokehome, J27 QWIIC_RA, J28 Pokehome, J29 Pokehome, J3 Pokehome, J30 Pokehome, J31 Pokehome, J32 Pokehome, J33 Pokehome, J34 Pokehome, J35 Pokehome, J36 QWIIC_RA, J37 Pokehome, J38 Pokehome, J39 Pokehome, J4 Pokehome, J40 Pokehome, J41 Pokehome, J42 Pokehome, J43 Pokehome, J44 Pokehome, J45 QWIIC_RA, J46 Pokehome, J47 Pokehome, J48 Pokehome, J49 Pokehome, J5 Pokehome, J50 Pokehome, J51 Pokehome, J52 Pokehome, J53 Pokehome, J54 QWIIC_RA, J6 Pokehome, J7 Pokehome, J8 Pokehome, J9 QWIIC_RA, U1 micro:bit, U2 micro:bit, U3 micro:bit, U4 micro:bit, U5 micro:bit, U6 micro:bit

Commit message: corrected panel to 1x5
previsously it was 1x6, so we wanted to keep it the same as before and good for pnp machines.
Parts:
- removed FD21, FD22, FD23, FD24: FIDUCIALUFIDUCIAL, SparkFun-Aesthetics:FIDUCIAL-MICRO
- removed H16, H17, H18: STAND-OFF, SparkFun-Hardware:STAND-OFF
- removed J46, J47, J48, J49, J50, J51, J52, J53: Pokehome, SparkFun-Connectors:1X02_POKEHOME
- removed J54: QWIIC_RA, SparkFun-Connectors:JST04_1MM_RA
- removed LOGO16: SFE_LOGO_FLAME.2_INCH, SparkFun-Aesthetics:SFE_LOGO_FLAME_.2
- removed LOGO17: OSHW-LOGOL, SparkFun-Aesthetics:OSHW-LOGO-L
- removed LOGO18: SFE_LOGO_NAME_FLAME.3_INCH, SparkFun-Aesthetics:SFE_LOGO_NAME_FLAME_.3
- removed R41, R42, R43, R44, R45, R46, R47, R48: 2.2k, SparkFun-Resistors:0603
- removed S31, S32, S33, S34, S35, S36: TACT, SparkFun-Switches:TACTILE_SWITCH_SMD_12MM
- removed TP66, TP67, TP68, TP69, TP70, TP71, TP72, TP73, TP74, TP75, TP76, TP77, TP78: TEST-POINT3X5, SparkFun-Connectors:PAD.03X.05
- removed U$16, U$17: LOGO-CONTROLBIT, SparkFun-Aesthetics:LOGO-CONTROLBIT
- removed U$18: (no value), SparkFun-Aesthetics:QWIIC_5MM
- removed U6: micro:bit, SparkFun-Connectors:MICRO:BIT-RA_SMD
- moved E$1 51.3 mm to (6.86, 258.1)
- moved E$2 51.3 mm to (6.86, 258.1)
- moved E$3 51.3 mm to (145.5, 258.1)
- moved E$4 51.3 mm to (145.5, 258.1)
Connections:
- removed net 3.3V5: J54.2, TP66.P$1, U6.P$27, U6.P$28, U6.P$29, U6.P$30, U6.P$31, U6.P$32
- removed net BTN_A5: R47.1, TP77.P$1, U6.P$7
- removed net BTN_B5: R48.1, TP74.P$1, U6.P$17
- removed net BTN_DN5: R44.1, TP75.P$1, U6.P$14
- removed net BTN_L5: R42.1, TP76.P$1, U6.P$10, U6.P$11, U6.P$12, U6.P$13
- removed net BTN_P10: R45.1, TP73.P$1, U6.P$18
- removed net BTN_P9: R46.1, TP71.P$1, U6.P$26
- removed net BTN_R5: R43.1, TP72.P$1, U6.P$19, U6.P$20, U6.P$21, U6.P$22
- removed net BTN_UP5: R41.1, TP78.P$1, U6.P$2, U6.P$3, U6.P$4, U6.P$5
- removed net GND5: J46.P1, J46.P3, J47.P1, J47.P3, J48.P1, J48.P3, J49.P1, J49.P3, J50.P1, J50.P3, J51.P1, J51.P3, J52.P1, J52.P3, J53.P1, J53.P3, J54.1, S31.1, S32.1, S33.3, S34.1, S35.1, S36.1, TP67.P$1, TP68.P$1, U6.P$35, U6.P$36, U6.P$37, U6.P$38, U6.P$39, U6.P$40
- removed net N$40: J46.P2, J46.P4, R41.2, S31.3
- removed net N$41: J49.P2, J49.P4, R42.2, S34.3
- removed net N$42: J48.P2, J48.P4, R44.2, S32.3
- removed net N$43: J47.P2, J47.P4, R43.2, S33.1
- removed net N$44: J50.P2, J50.P4, R45.2, S35.3
- removed net N$45: J51.P2, J51.P4, R46.2, S36.3
- removed net N$46: J52.P2, J52.P4, R47.2
- removed net N$47: J53.P2, J53.P4, R48.2
- removed net SCL5: J54.4, TP70.P$1, U6.P$33
- removed net SDA5: J54.3, TP69.P$1, U6.P$34
Routing:
- net 3.3V5: track 117.8 -> 0.00 mm, vias 2 -> 0
- net SCL5: track 101.7 -> 0.00 mm, vias 2 -> 0
- net SDA5: track 95.3 -> 0.00 mm, vias 2 -> 0
- net N$40: track 79.1 -> 0.00 mm, vias 2 -> 0
- net BTN_P9: track 71.6 -> 0.00 mm, vias 1 -> 0
- net BTN_R5: track 71.5 -> 0.00 mm, vias 1 -> 0
- net BTN_P10: track 70.7 -> 0.00 mm, vias 1 -> 0
- net BTN_B5: track 69.7 -> 0.00 mm, vias 1 -> 0
- net BTN_A5: track 64.3 -> 0.00 mm, vias 1 -> 0
- net N$41: track 61.5 -> 0.00 mm, vias 2 -> 0
- net GND5: track 55.5 -> 0.00 mm, vias 51 -> 0
- net BTN_L5: track 53.8 -> 0.00 mm, vias 1 -> 0
- net N$44: track 52.0 -> 0.00 mm, vias 1 -> 0
- net BTN_DN5: track 50.1 -> 0.00 mm, vias 1 -> 0
- net N$45: track 48.7 -> 0.00 mm, vias 1 -> 0
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- removed copper zone on layer 1, net GND5
- removed copper zone on layer 16, net GND5
Other:
- board size 172.5 x 327.4 mm -> 172.5 x 276.1 mm
